File: ESC_PCB/ESC_3S/ESC_3S.kicad_sch (KiCad schematic)
At the start: 11 parts, among them U1 MIC5219-3.3YM5, U2 MP2359

Commit message: add .ioc and temperature done sch
Parts:
- removed C1: 22pF 25V, Capacitor_SMD:C_0603_1608Metric_Pad1.08x0.95mm_HandSolder, symbol Device:C
- removed C2: 10nF 50V, Capacitor_SMD:C_0603_1608Metric_Pad1.08x0.95mm_HandSolder, symbol Device:C
- removed C3: C, Capacitor_SMD:C_0603_1608Metric_Pad1.08x0.95mm_HandSolder, symbol Device:C
- removed C4: 22uF 6.3V, Capacitor_SMD:C_0805_2012Metric_Pad1.18x1.45mm_HandSolder, symbol Device:C
- removed C5: 2.2uF 16V, Capacitor_SMD:C_1206_3216Metric_Pad1.33x1.80mm_HandSolder, symbol Device:C
- removed C6: 470pF, Capacitor_SMD:C_0603_1608Metric_Pad1.08x0.95mm_HandSolder, symbol Device:C
- removed L1: 4.7uH, Inductor_SMD:L_0805_2012Metric_Pad1.05x1.20mm_HandSolder, symbol Device:L
- removed R1: 52.3K, symbol Device:R
- removed R2: 10K, symbol Device:R
- removed U1: MIC5219-3.3YM5, Package_TO_SOT_SMD:SOT-23-5, symbol Regulator_Linear:MIC5219-3.3YM5
- removed U2: MP2359, easyeda2kicad:SOT-23-6_L2.9-W1.6-P0.95-LS2.8-BR, symbol easyeda2kicad:MP2359DJ-LF-Z-MS
Other:
- added sheet Addition (untitled.kicad_sch)
- added sheet Gate Driver and 3PH Inverter Bridge (IVT.kicad_sch)
- added sheet MCU Section (MCUSection.kicad_sch)
- added sheet Power (Power ESC.kicad_sch)
- note removed: "BUCK BAT TO 5V"
- note removed: "LDO 3v3"

Commit message: done schematic
Other:
- sheet Addition ports: added CAN_RX, CAN_TX, Temperature_fed, VBAT_SENS; removed none
- sheet Gate Driver and 3PH Inverter Bridge ports: added Curr_fdbk1_OPAmp+, Curr_fdbk1_OPAmp-, Curr_fdbk2_OPAmp+, Curr_fdbk2_OPAmp-, Curr_fdbk3_OPAmp+, Curr_fdbk3_OPAmp-; removed none
- sheet MCU Section ports: added CAN_RX, CAN_TX, Curr_fdbk1_OPAmp+, Curr_fdbk1_OPAmp-, Curr_fdbk2_OPAmp+, Curr_fdbk2_OPAmp-, Curr_fdbk3_OPAmp+, Curr_fdbk3_OPAmp-, Temperature_fed, VBAT_SENS; removed none
