File: ESC_PCB/ESC_3S/Power ESC.kicad_sch (KiCad schematic)
At the start: 28 parts, among them J2 Conn_01x01_Pin, J3 Conn_01x01_Pin, U1 MIC5219-3.3YM5, U2 MP2359

Commit message: done schematic
Parts:
- J2, J3: footprint (none) -> Connector_Wire:SolderWire-0.25sqmm_1x01_D0.65mm_OD1.7mm
- R1, R2: footprint (none) -> Resistor_SMD:R_0603_1608Metric_Pad0.98x0.95mm_HandSolder
Changed lines of the file:
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@@
 			)
 		)
-		(property "Footprint" ""
+		(property "Footprint" "Resistor_SMD:R_0603_1608Metric_Pad0.98x0.95mm_HandSolder"
 			(at 113.792 127 90)
 			(effects
@@
 			)
 		)
-		(property "Footprint" ""
+		(property "Footprint" "Connector_Wire:SolderWire-0.25sqmm_1x01_D0.65mm_OD1.7mm"
 			(at 82.55 55.88 0)
 			(effects
@@
 			)
 		)
-		(property "Footprint" ""
+		(property "Footprint" "Resistor_SMD:R_0603_1608Metric_Pad0.98x0.95mm_HandSolder"
 			(at 113.792 138.43 90)
 			(effects
@@
 			)
 		)
-		(property "Footprint" ""
+		(property "Footprint" "Connector_Wire:SolderWire-0.25sqmm_1x01_D0.65mm_OD1.7mm"
 			(at 82.55 43.18 0)
 			(effects
