File: ESC_PCB/ESC_3S/Power ESC.kicad_sch (KiCad schematic)
At the start: 30 parts, among them J2 Conn_01x01_Pin, J3 Conn_01x01_Pin, U2 MP2359, U7 LD1117S33TR_SOT223

Commit message: xuat gerber done
Changed lines of the file:
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@@
 		(color 0 0 0 0)
+	)
+	(bus_entry
+		(at 86.36 46.99)
+		(size 2.54 2.54)
+		(stroke
+			(width 0)
+			(type default)
+		)
 	)
 	(wire
