File: ESC_PCB/ESC_3S/MCUSection.kicad_sch (KiCad schematic)
At the start: 21 parts, among them J1 DEBUG&FLASH, J5 UART, U3 STM32G431CBUx, X1 Q13FC1350000400, X2 X50328MSB2GI

Commit message: add .ioc and temperature done sch
Connections:
- net Curr_fdbk3_OPAmp+: now reaches U3.17 (PB0)
- net Curr_fdbk3_OPAmp-: now reaches U3.19 (PB2)
Changed lines of the file:
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@@
+		)
+	)
+	(hierarchical_label "Curr_fdbk3_OPAmp-"
+		(shape input)
+		(at 203.2 100.33 180)
+		(effects
+			(font
+				(size 1.27 1.27)
+				(thickness 0.254)
+				(bold yes)
+			)
+			(justify right)
 		)
 	)
@@
 		(effects
 			(font
+				(size 1.27 1.27)
+				(thickness 0.254)
+				(bold yes)
+			)
+			(justify right)
+		)
+	)
+	(hierarchical_label "Curr_fdbk3_OPAmp+"
+		(shape input)
+		(at 203.2 95.25 180)
+		(effects
+			(font

Commit message: done schematic
Parts:
- C10, C8: footprint (none) -> Capacitor_SMD:C_0603_1608Metric_Pad1.08x0.95mm_HandSolder
Connections:
- net GND: now also C12.2, C13.2, C14.2, C15.2, C16.2, C17.2
- net VBAT_SENS: now reaches U3.8 (PA0)
- no-connect marks 0 -> 15
Other:
- moved on the sheet: C12, C13, C14, C15, C16, C17, FB1, J1, J5

Commit message: dang layout
Changed lines of the file:
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@@
 	(wire
 		(pts
+			(xy 193.04 100.33) (xy 203.2 100.33)
+		)
+		(stroke
+			(width 0)
+			(type default)
+		)
+	)
+	(wire
+		(pts
 			(xy 74.93 142.24) (xy 74.93 146.05)
 		)
@@
 	(wire
 		(pts
-			(xy 238.76 82.55) (xy 245.11 82.55)
+			(xy 238.76 82.55) (xy 252.73 82.55)
 		)
 		(stroke
@@
 	(wire
 		(pts
-			(xy 238.76 77.47) (xy 245.11 77.47)
+			(xy 238.76 77.47) (xy 252.73 77.47)
 		)
 		(stroke
@@
 	(wire
 		(pts
-			(xy 191.77 57.15) (xy 203.2 57.15)
+			(xy 193.04 57.15) (xy 203.2 57.15)
 		)
 		(stroke
@@
 	(wire
 		(pts
-			(xy 191.77 62.23) (xy 203.2 62.23)
+			(xy 193.04 62.23) (xy 203.2 62.23)
 		)
 		(stroke
@@
 	(wire
 		(pts
-			(xy 238.76 80.01) (xy 245.11 80.01)
+			(xy 238.76 80.01) (xy 252.73 80.01)
 		)
 		(stroke
@@
 	(wire
 		(pts
-			(xy 245.11 59.69) (xy 238.76 59.69)
+			(xy 252.73 59.69) (xy 238.76 59.69)
 		)
 		(stroke
@@
 	(wire
 		(pts
-			(xy 238.76 85.09) (xy 245.11 85.09)
+			(xy 238.76 85.09) (xy 252.73 85.09)
 		)
 		(stroke
@@
 	(wire
 		(pts
-			(xy 245.11 74.93) (xy 238.76 74.93)
+			(xy 252.73 74.93) (xy 238.76 74.93)
 		)
 		(stroke
@@
 	(wire
 		(pts
-			(xy 238.76 87.63) (xy 245.11 87.63)
+			(xy 238.76 87.63) (xy 252.73 87.63)
 		)
 		(stroke
@@
 	(wire
 		(pts
-			(xy 245.11 64.77) (xy 238.76 64.77)
+			(xy 252.73 64.77) (xy 238.76 64.77)
 		)
 		(stroke
@@
 	(wire
 		(pts
-			(xy 245.11 57.15) (xy 238.76 57.15)
+			(xy 252.73 57.15) (xy 238.76 57.15)
 		)
 		(stroke
@@
 	(wire
 		(pts
+			(xy 193.04 95.25) (xy 203.2 95.25)
+		)
+		(stroke
+			(width 0)
+			(type default)
+		)
+	)
+	(wire
+		(pts
 			(xy 149.86 43.18) (xy 149.86 49.53)
 		)
@@
 	(wire
 		(pts
-			(xy 245.11 69.85) (xy 238.76 69.85)
+			(xy 252.73 69.85) (xy 238.76 69.85)
 		)
 		(stroke
@@
 	)
 	(label "RST"
-		(at 191.77 62.23 0)
+		(at 193.04 62.23 0)
 		(effects
 			(font
@@
 	)
 	(label "VREF"
-		(at 191.77 57.15 0)
+		(at 193.04 57.15 0)
 		(effects
 			(font
@@
 	(hierarchical_label "Curr_fdbk3_OPAmp-"
 		(shape input)
-		(at 203.2 100.33 180)
+		(at 193.04 100.33 180)
 		(effects
 			(font
@@
 	(hierarchical_label "TIM1_CH2N"
 		(shape input)
-		(at 245.11 87.63 0)
+		(at 252.73 87.63 0)
 		(effects
 			(font
@@
 	(hierarchical_label "Curr_fdbk1_OPAmp-"
 		(shape input)
-		(at 245.11 64.77 0)
+		(at 252.73 64.77 0)
 		(effects
 			(font
@@
 	(hierarchical_label "Curr_fdbk3_OPAmp+"
 		(shape input)
-		(at 203.2 95.25 180)
+		(at 193.04 95.25 180)
 		(effects
 			(font
@@
 	(hierarchical_label "TIM1_CH1"
 		(shape input)
-		(at 245.11 77.47 0)
+		(at 252.73 77.47 0)
 		(effects
 			(font
@@
 	(hierarchical_label "Curr_fdbk1_OPAmp+"
 		(shape input)
-		(at 245.11 59.69 0)
+		(at 252.73 59.69 0)
 		(effects
 			(font
@@
 	(hierarchical_label "CAN_RX"
 		(shape input)
-		(at 245.11 85.09 0)
+		(at 252.73 85.09 0)
 		(effects
 			(font
@@
 	(hierarchical_label "VBAT_SENS"
 		(shape input)
-		(at 245.11 57.15 0)
+		(at 252.73 57.15 0)
 		(effects
 			(font
@@
 	(hierarchical_label "TIM1_CH2"
 		(shape input)
-		(at 245.11 80.01 0)
+		(at 252.73 80.01 0)
 		(effects
 			(font
@@
 	(hierarchical_label "Curr_fdbk2_OPAmp+"
 		(shape input)
-		(at 245.11 69.85 0)
+		(at 252.73 69.85 0)
 		(effects
 			(font
@@
 	(hierarchical_label "Curr_fdbk2_OPAmp-"
 		(shape input)
-		(at 245.11 74.93 0)
+		(at 252.73 74.93 0)
 		(effects
 			(font
@@
 	(hierarchical_label "TIM1_CH3"
 		(shape input)
-		(at 245.11 82.55 0)
+		(at 252.73 82.55 0)
 		(effects
 			(font
@@
 		)
 		(instances
-			(project ""
+			(project "ESC_3S"
 				(path "/66ec60ca-6d64-4483-97f1-d2d066c965b7/9bfba7c7-25d8-4f24-9954-d47ed221637e"
 					(reference "#PWR08")
@@
 		)
 		(instances
-			(project ""
+			(project "ESC_3S"
 				(path "/66ec60ca-6d64-4483-97f1-d2d066c965b7/9bfba7c7-25d8-4f24-9954-d47ed221637e"
 					(reference "C12")
@@
 		)
 		(instances
-			(project ""
+			(project "ESC_3S"
 				(path "/66ec60ca-6d64-4483-97f1-d2d066c965b7/9bfba7c7-25d8-4f24-9954-d47ed221637e"
 					(reference "S1")
@@
 		)
 		(instances
-			(project ""
+			(project "ESC_3S"
 				(path "/66ec60ca-6d64-4483-97f1-d2d066c965b7/9bfba7c7-25d8-4f24-9954-d47ed221637e"
 					(reference "#PWR016")
@@
 		)
 		(instances
-			(project ""
+			(project "ESC_3S"
 				(path "/66ec60ca-6d64-4483-97f1-d2d066c965b7/9bfba7c7-25d8-4f24-9954-d47ed221637e"
 					(reference "J1")
@@
 		)
 		(instances
-			(project ""
+			(project "ESC_3S"
 				(path "/66ec60ca-6d64-4483-97f1-d2d066c965b7/9bfba7c7-25d8-4f24-9954-d47ed221637e"
 					(reference "FB1")
@@
 		)
 		(instances
-			(project ""
+			(project "ESC_3S"
 				(path "/66ec60ca-6d64-4483-97f1-d2d066c965b7/9bfba7c7-25d8-4f24-9954-d47ed221637e"
 					(reference "#PWR012")
@@
 		)
 		(instances
-			(project ""
+			(project "ESC_3S"
 				(path "/66ec60ca-6d64-4483-97f1-d2d066c965b7/9bfba7c7-25d8-4f24-9954-d47ed221637e"
 					(reference "U3")
@@
 		)
 		(instances
-			(project ""
+			(project "ESC_3S"
 				(path "/66ec60ca-6d64-4483-97f1-d2d066c965b7/9bfba7c7-25d8-4f24-9954-d47ed221637e"
 					(reference "#PWR014")
@@
 		)
 		(instances
-			(project ""
+			(project "ESC_3S"
 				(path "/66ec60ca-6d64-4483-97f1-d2d066c965b7/9bfba7c7-25d8-4f24-9954-d47ed221637e"
 					(reference "#PWR020")
@@
 		)
 		(instances
-			(project ""
+			(project "ESC_3S"
 				(path "/66ec60ca-6d64-4483-97f1-d2d066c965b7/9bfba7c7-25d8-4f24-9954-d47ed221637e"
 					(reference "R4")
@@
 		)
 		(instances
-			(project ""
+			(project "ESC_3S"
 				(path "/66ec60ca-6d64-4483-97f1-d2d066c965b7/9bfba7c7-25d8-4f24-9954-d47ed221637e"
 					(reference "#PWR059")
@@
 		)
 		(instances
-			(project ""
+			(project "ESC_3S"
 				(path "/66ec60ca-6d64-4483-97f1-d2d066c965b7/9bfba7c7-25d8-4f24-9954-d47ed221637e"
 					(reference "#PWR011")
@@
 		)
 		(instances
-			(project ""
+			(project "ESC_3S"
 				(path "/66ec60ca-6d64-4483-97f1-d2d066c965b7/9bfba7c7-25d8-4f24-9954-d47ed221637e"
 					(reference "#PWR019")
@@
 		)
 		(instances
-			(project ""
+			(project "ESC_3S"
 				(path "/66ec60ca-6d64-4483-97f1-d2d066c965b7/9bfba7c7-25d8-4f24-9954-d47ed221637e"
 					(reference "R3")
@@
 		)
 		(instances
-			(project ""
+			(project "ESC_3S"
 				(path "/66ec60ca-6d64-4483-97f1-d2d066c965b7/9bfba7c7-25d8-4f24-9954-d47ed221637e"
 					(reference "C11")
@@
 		)
 		(instances
-			(project ""
+			(project "ESC_3S"
 				(path "/66ec60ca-6d64-4483-97f1-d2d066c965b7/9bfba7c7-25d8-4f24-9954-d47ed221637e"
 					(reference "#PWR018")

Commit message: layout
Parts:
- removed J1: DEBUG&FLASH, Connector_PinHeader_2.54mm:PinHeader_1x05_P2.54mm_Vertical, symbol Connector:Conn_01x05_Pin
- added J4: Flash&Debug, Connector_PinHeader_1.27mm:PinHeader_1x04_P1.27mm_Vertical, symbol Connector_Generic:Conn_01x04
Connections:
- net GND: now also J4.1 (Pin_1)
- net SWCLK: now also J4.3 (Pin_3)
- net SWDIO: now also J4.2 (Pin_2)
- net SWO: now also J4.4 (Pin_4)
Changed lines of the file:
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@@
 	)
 	(junction
+		(at 143.51 60.96)
+		(diameter 0)
+		(color 0 0 0 0)
+	)
+	(junction
 		(at 38.1 54.61)
 		(diameter 0)
@@
 	)
 	(junction
+		(at 151.13 63.5)
+		(diameter 0)
+		(color 0 0 0 0)
+	)
+	(junction
 		(at 80.01 88.9)
 		(diameter 0)
@@
 	(wire
 		(pts
+			(xy 142.24 60.96) (xy 143.51 60.96)
+		)
+		(stroke
+			(width 0)
+			(type default)
+		)
+	)
+	(wire
+		(pts
 			(xy 38.1 54.61) (xy 38.1 57.15)
 		)
@@
 	(wire
 		(pts
-			(xy 139.7 57.15) (xy 147.32 57.15)
+			(xy 151.13 55.88) (xy 143.51 55.88)
 		)
 		(stroke
@@
 	(wire
 		(pts
-			(xy 139.7 52.07) (xy 147.32 52.07)
-		)
-		(stroke
-			(width 0)
-			(type default)
-		)
-	)
-	(wire
-		(pts
 			(xy 102.87 91.44) (xy 102.87 88.9)
 		)
@@
 	(wire
 		(pts
-			(xy 139.7 54.61) (xy 147.32 54.61)
+			(xy 151.13 58.42) (xy 143.51 58.42)
 		)
 		(stroke
@@
 	(wire
 		(pts
+			(xy 143.51 60.96) (xy 151.13 60.96)
+		)
+		(stroke
+			(width 0)
+			(type default)
+		)
+	)
+	(wire
+		(pts
 			(xy 114.3 139.7) (xy 114.3 142.24)
 		)
@@
 	(wire
 		(pts
-			(xy 139.7 49.53) (xy 149.86 49.53)
+			(xy 151.13 53.34) (xy 143.51 53.34)
 		)
 		(stroke
@@
 	(wire
 		(pts
-			(xy 139.7 59.69) (xy 147.32 59.69)
+			(xy 218.44 45.72) (xy 220.98 45.72)
 		)
 		(stroke
@@
 	(wire
 		(pts
-			(xy 218.44 45.72) (xy 220.98 45.72)
+			(xy 100.33 55.88) (xy 90.17 55.88)
 		)
 		(stroke
@@
 	(wire
 		(pts
-			(xy 100.33 55.88) (xy 90.17 55.88)
+			(xy 90.17 55.88) (xy 90.17 60.96)
 		)
 		(stroke
@@
 	(wire
 		(pts
-			(xy 90.17 55.88) (xy 90.17 60.96)
+			(xy 48.26 54.61) (xy 38.1 54.61)
 		)
 		(stroke
@@
 	(wire
 		(pts
-			(xy 48.26 54.61) (xy 38.1 54.61)
+			(xy 59.69 88.9) (xy 64.77 88.9)
 		)
 		(stroke
@@
 	(wire
 		(pts
-			(xy 59.69 88.9) (xy 64.77 88.9)
+			(xy 151.13 60.96) (xy 151.13 63.5)
 		)
 		(stroke
@@
 	(wire
 		(pts
-			(xy 149.86 43.18) (xy 149.86 49.53)
+			(xy 151.13 63.5) (xy 149.86 63.5)
 		)
 		(stroke
@@
 		)
 	)
-	(label "SWCLK"
-		(at 140.97 57.15 0)
-		(effects
-			(font
-				(size 1.27 1.27)
-			)
-			(justify left bottom)
-		)
-	)
 	(label "OSC32_IN"
 		(at 193.04 87.63 0)
@@
 		)
 	)
-	(label "SWDIO"
-		(at 140.97 54.61 0)
-		(effects
-			(font
-				(size 1.27 1.27)
-			)
-			(justify left bottom)
-		)
-	)
 	(label "RX"
 		(at 193.04 113.03 0)
@@
 		)
 	)
+	(label "SWO"
+		(at 151.13 53.34 180)
+		(effects
+			(font
+				(size 1.27 1.27)
+			)
+			(justify right bottom)
+		)
+	)
+	(label "SWCLK"
+		(at 151.13 55.88 180)
+		(effects
+			(font
+				(size 1.27 1.27)
+			)
+			(justify right bottom)
+		)
+	)
 	(label "OSC_OUT"
 		(at 193.04 69.85 0)
@@
 		)
 	)
-	(label "SWO"
-		(at 143.51 59.69 0)
+	(label "BOOT0"
+		(at 193.04 115.57 0)
 		(effects
 			(font
@@
 		)
 	)
-	(label "BOOT0"
-		(at 193.04 115.57 0)
+	(label "SWDIO"
+		(at 151.13 58.42 180)
 		(effects
 			(font
 				(size 1.27 1.27)
 			)
-			(justify left bottom)
+			(justify right bottom)
 		)
 	)
@@
 	(symbol
 		(lib_id "power:GND")
-		(at 147.32 52.07 90)
+		(at 151.13 63.5 0)
 		(unit 1)
 		(exclude_from_sim no)
@@
 		(on_board yes)
 		(dnp no)
-		(fields_autoplaced yes)
 		(property "Reference" "#PWR016"
-			(at 153.67 52.07 0)
+			(at 151.13 69.85 0)
 			(effects
 				(font
@@
 		)
 		(property "Value" "GND"
-			(at 151.13 52.0699 90)
+			(at 151.1301 67.31 90)
 			(effects
 				(font
@@
 		)
 		(property "Footprint" ""
-			(at 147.32 52.07 0)
+			(at 151.13 63.5 0)
 			(effects
 				(font
@@
 		)
 		(property "Datasheet" ""
-			(at 147.32 52.07 0)
+			(at 151.13 63.5 0)
 			(effects
 				(font
@@
 		)
 		(property "Description" "Power symbol creates a global label with name \"GND\" , ground"
-			(at 147.32 52.07 0)
+			(at 151.13 63.5 0)
 			(effects
 				(font
@@
 	)
 	(symbol
-		(lib_id "Connector:Conn_01x05_Pin")
-		(at 134.62 54.61 0)
-		(unit 1)
-		(exclude_from_sim no)
-		(in_bom yes)
-		(on_board yes)
-		(dnp no)
-		(fields_autoplaced yes)
-		(property "Reference" "J1"
-			(at 135.255 44.45 0)
-			(effects
-				(font
-					(size 1.27 1.27)
-				)
-			)
-		)
-		(property "Value" "DEBUG&FLASH"
-			(at 135.255 46.99 0)
-			(effects
-				(font
-					(size 1.27 1.27)
-				)
-			)
-		)
-		(property "Footprint" "Connector_PinHeader_2.54mm:PinHeader_1x05_P2.54mm_Vertical"
-			(at 134.62 54.61 0)
-			(effects
-				(font
-					(size 1.27 1.27)
-				)
-				(hide yes)
-			)
-		)
-		(property "Datasheet" "~"
-			(at 134.62 54.61 0)
-			(effects
-				(font
-					(size 1.27 1.27)
-				)
-				(hide yes)
-			)
-		)
-		(property "Description" "Generic connector, single row, 01x05, script generated"
-			(at 134.62 54.61 0)
-			(effects
-				(font
-					(size 1.27 1.27)
-				)
-				(hide yes)
-			)
-		)
-		(pin "2"
-		)
-		(pin "1"
-		)
-		(pin "5"
-		)
-		(pin "3"
-		)
-		(pin "4"
-		)
-		(instances
-			(project "ESC_3S"
-				(path "/66ec60ca-6d64-4483-97f1-d2d066c965b7/9bfba7c7-25d8-4f24-9954-d47ed221637e"
-					(reference "J1")
-					(unit 1)
-				)
-			)
-		)
-	)
-	(symbol
 		(lib_id "Device:C")
 		(at 59.69 95.25 0)
@@
 	)
 	(symbol
-		(lib_id "power:+3.3V")
-		(at 149.86 43.18 0)
+		(lib_id "power:GND")
+		(at 74.93 59.69 0)
 		(unit 1)
 		(exclude_from_sim no)
@@
 		(dnp no)
 		(fields_autoplaced yes)
-		(property "Reference" "#PWR015"
-			(at 149.86 46.99 0)
+		(property "Reference" "#PWR014"
+			(at 74.93 66.04 0)
 			(effects
 				(font
@@
 			)
 		)
-		(property "Value" "+3.3V"
-			(at 149.86 38.1 0)
+		(property "Value" "GND"
+			(at 74.93 64.77 0)
 			(effects
 				(font
@@
 		)
 		(property "Footprint" ""
-			(at 149.86 43.18 0)
+			(at 74.93 59.69 0)
 			(effects
 				(font
@@
 		)
 		(property "Datasheet" ""
-			(at 149.86 43.18 0)
+			(at 74.93 59.69 0)
 			(effects
 				(font
@@
 			)
 		)
-		(property "Description" "Power symbol creates a global label with name \"+3.3V\""
-			(at 149.86 43.18 0)
+		(property "Description" "Power symbol creates a global label with name \"GND\" , ground"
+			(at 74.93 59.69 0)
 			(effects
 				(font
@@
 			(project "ESC_3S"
 				(path "/66ec60ca-6d64-4483-97f1-d2d066c965b7/9bfba7c7-25d8-4f24-9954-d47ed221637e"
-					(reference "#PWR015")
+					(reference "#PWR014")
 					(unit 1)
 				)
@@
 	)
 	(symbol
-		(lib_id "power:GND")
-		(at 74.93 59.69 0)
+		(lib_id "Connector_Generic:Conn_01x04")
+		(at 138.43 58.42 180)
 		(unit 1)
 		(exclude_from_sim no)
@@
 		(dnp no)
 		(fields_autoplaced yes)
-		(property "Reference" "#PWR014"
-			(at 74.93 66.04 0)
+		(property "Reference" "J4"
+			(at 138.43 46.99 0)
 			(effects
 				(font
 					(size 1.27 1.27)
 				)
-				(hide yes)
 			)
 		)
-		(property "Value" "GND"
-			(at 74.93 64.77 0)
+		(property "Value" "Flash&Debug"
+			(at 138.43 49.53 0)
 			(effects
 				(font
@@
 			)
 		)
-		(property "Footprint" ""
-			(at 74.93 59.69 0)
+		(property "Footprint" "Connector_PinHeader_1.27mm:PinHeader_1x04_P1.27mm_Vertical"
+			(at 138.43 58.42 0)
 			(effects
 				(font
@@
 			)
 		)
-		(property "Datasheet" ""
-			(at 74.93 59.69 0)
+		(property "Datasheet" "~"
+			(at 138.43 58.42 0)
 			(effects
 				(font
@@
 			)
 		)
-		(property "Description" "Power symbol creates a global label with name \"GND\" , ground"
-			(at 74.93 59.69 0)
+		(property "Description" "Generic connector, single row, 01x04, script generated (kicad-library-utils/schlib/autogen/connector/)"
+			(at 138.43 58.42 0)
 			(effects
 				(font
@@
 			)
 		)
+		(pin "2"
+		)
+		(pin "4"
+		)
 		(pin "1"
 		)
+		(pin "3"
+		)
 		(instances
 			(project "ESC_3S"
 				(path "/66ec60ca-6d64-4483-97f1-d2d066c965b7/9bfba7c7-25d8-4f24-9954-d47ed221637e"
-					(reference "#PWR014")
+					(reference "J4")
 					(unit 1)
 				)
