File: ESC_PCB/ESC_3S/IVT.kicad_sch (KiCad schematic)
At the start: 45 parts, among them Q1 CSD18532Q5BT, Q2 CSD18532Q5BT, Q3 CSD18532Q5BT, Q4 CSD18532Q5BT, Q5 CSD18532Q5BT, Q6 CSD18532Q5BT, U4 FD6288Q

Commit message: add .ioc and temperature done sch
Parts:
- added JP3: SolderJumper_2_Open, Jumper:SolderJumper-2_P1.3mm_Open_TrianglePad1.0x1.5mm, symbol Jumper:SolderJumper_2_Open
- added R35: 0.001R, Resistor_SMD:R_2512_6332Metric_Pad1.40x3.35mm_HandSolder, symbol Device:R
- added R36: 22K, Resistor_SMD:R_0603_1608Metric_Pad0.98x0.95mm_HandSolder, symbol Device:R
- added R37: 2.2K, Resistor_SMD:R_0603_1608Metric_Pad0.98x0.95mm_HandSolder, symbol Device:R
- added R38: 1.5K, Resistor_SMD:R_0603_1608Metric_Pad0.98x0.95mm_HandSolder, symbol Device:R
- R25, R27: value 22K -> 2.2K
Connections:
- net +3.3V: now also R36.1
- net GND: now also JP3.2 (B), R35.2, R37.2
- net Phase_3 renamed V_Shunt_3+
- net V_Shunt_3+: now also R35.1, R38.2
- new net Curr_fdbk3_OPAmp+: R36.2, R37.1, R38.1
- new net Curr_fdbk3_OPAmp-: JP3.1 (A)
Other:
- moved on the sheet: C18, C19, C20, C21, C36, C37, C38, C39, C40, C41, D2, D3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

Commit message: done schematic
Parts:
- added J6: U, Connector_Wire:SolderWirePad_1x01_SMD_1x2mm, symbol Connector:Conn_01x01_Pin
- added J7: V, Connector_Wire:SolderWirePad_1x01_SMD_1x2mm, symbol Connector:Conn_01x01_Pin
- added J8: W, Connector_Wire:SolderWirePad_1x01_SMD_1x2mm, symbol Connector:Conn_01x01_Pin
Connections:
- net GND: now also U4.25 (EP)
- net Phase_1: now also J6.1 (Pin_1)
- net Phase_2: now also J7.1 (Pin_1)
- net V_Shunt_3+: now also Q6.1 (S), Q6.2 (S), Q6.3 (S), R18.2; no longer C41.1, Q5.1 (S), Q5.2 (S), Q5.3 (S), Q6.5 (D), Q6.6 (D), Q6.7 (D), Q6.8 (D), Q6.9 (D), R17.2, R19.1, U4.12 (VS3)
- new net Phase_3: C41.1, J8.1 (Pin_1), Q5.1 (S), Q5.2 (S), Q5.3 (S), Q6.5 (D), Q6.6 (D), Q6.7 (D), Q6.8 (D), Q6.9 (D), R17.2, R19.1, U4.12 (VS3)
Other:
- moved on the sheet: R38

Commit message: dang layout
Changed lines of the file:
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@@
 	(paper "A4")
 	(rectangle
-		(start 115.57 80.01)
+		(start 114.3 80.01)
 		(end 280.67 157.48)
 		(stroke
@@
 		)
 		(instances
-			(project ""
+			(project "ESC_3S"
 				(path "/66ec60ca-6d64-4483-97f1-d2d066c965b7/a3efd6b8-4fcd-4591-95ab-0bc4985f625a"
 					(reference "C39")
@@
 		)
 		(instances
-			(project ""
+			(project "ESC_3S"
 				(path "/66ec60ca-6d64-4483-97f1-d2d066c965b7/a3efd6b8-4fcd-4591-95ab-0bc4985f625a"
 					(reference "C36")
@@
 		)
 		(instances
-			(project ""
+			(project "ESC_3S"
 				(path "/66ec60ca-6d64-4483-97f1-d2d066c965b7/a3efd6b8-4fcd-4591-95ab-0bc4985f625a"
 					(reference "#PWR040")
@@
 		)
 		(instances
-			(project ""
+			(project "ESC_3S"
 				(path "/66ec60ca-6d64-4483-97f1-d2d066c965b7/a3efd6b8-4fcd-4591-95ab-0bc4985f625a"
 					(reference "U4")
@@
 		)
 		(instances
-			(project ""
+			(project "ESC_3S"
 				(path "/66ec60ca-6d64-4483-97f1-d2d066c965b7/a3efd6b8-4fcd-4591-95ab-0bc4985f625a"
 					(reference "J6")
@@
 		)
 		(instances
-			(project ""
+			(project "ESC_3S"
 				(path "/66ec60ca-6d64-4483-97f1-d2d066c965b7/a3efd6b8-4fcd-4591-95ab-0bc4985f625a"
 					(reference "#PWR035")
@@
 		)
 		(instances
-			(project ""
+			(project "ESC_3S"
 				(path "/66ec60ca-6d64-4483-97f1-d2d066c965b7/a3efd6b8-4fcd-4591-95ab-0bc4985f625a"
 					(reference "Q1")
@@
 		)
 		(instances
-			(project ""
+			(project "ESC_3S"
 				(path "/66ec60ca-6d64-4483-97f1-d2d066c965b7/a3efd6b8-4fcd-4591-95ab-0bc4985f625a"
 					(reference "#PWR058")
@@
 		)
 		(instances
-			(project ""
+			(project "ESC_3S"
 				(path "/66ec60ca-6d64-4483-97f1-d2d066c965b7/a3efd6b8-4fcd-4591-95ab-0bc4985f625a"
 					(reference "C18")
@@
 		)
 		(instances
-			(project ""
+			(project "ESC_3S"
 				(path "/66ec60ca-6d64-4483-97f1-d2d066c965b7/a3efd6b8-4fcd-4591-95ab-0bc4985f625a"
 					(reference "R5")
@@
 		)
 		(instances
-			(project ""
+			(project "ESC_3S"
 				(path "/66ec60ca-6d64-4483-97f1-d2d066c965b7/a3efd6b8-4fcd-4591-95ab-0bc4985f625a"
 					(reference "R20")
@@
 		)
 		(instances
-			(project ""
+			(project "ESC_3S"
 				(path "/66ec60ca-6d64-4483-97f1-d2d066c965b7/a3efd6b8-4fcd-4591-95ab-0bc4985f625a"
 					(reference "#PWR022")
@@
 		)
 		(instances
-			(project ""
+			(project "ESC_3S"
 				(path "/66ec60ca-6d64-4483-97f1-d2d066c965b7/a3efd6b8-4fcd-4591-95ab-0bc4985f625a"
 					(reference "D2")
@@
 		)
 		(instances
-			(project ""
+			(project "ESC_3S"
 				(path "/66ec60ca-6d64-4483-97f1-d2d066c965b7/a3efd6b8-4fcd-4591-95ab-0bc4985f625a"
 					(reference "#PWR027")
@@
 		)
 		(instances
-			(project ""
+			(project "ESC_3S"
 				(path "/66ec60ca-6d64-4483-97f1-d2d066c965b7/a3efd6b8-4fcd-4591-95ab-0bc4985f625a"
 					(reference "R9")
@@
 		)
 		(instances
-			(project ""
+			(project "ESC_3S"
 				(path "/66ec60ca-6d64-4483-97f1-d2d066c965b7/a3efd6b8-4fcd-4591-95ab-0bc4985f625a"
 					(reference "#PWR028")
@@
 		)
 		(instances
-			(project ""
+			(project "ESC_3S"
 				(path "/66ec60ca-6d64-4483-97f1-d2d066c965b7/a3efd6b8-4fcd-4591-95ab-0bc4985f625a"
 					(reference "#PWR033")
@@
 		)
 		(instances
-			(project ""
+			(project "ESC_3S"
 				(path "/66ec60ca-6d64-4483-97f1-d2d066c965b7/a3efd6b8-4fcd-4591-95ab-0bc4985f625a"
 					(reference "R22")
@@
 		)
 		(instances
-			(project ""
+			(project "ESC_3S"
 				(path "/66ec60ca-6d64-4483-97f1-d2d066c965b7/a3efd6b8-4fcd-4591-95ab-0bc4985f625a"
 					(reference "#PWR021")
@@
 		)
 		(instances
-			(project ""
+			(project "ESC_3S"
 				(path "/66ec60ca-6d64-4483-97f1-d2d066c965b7/a3efd6b8-4fcd-4591-95ab-0bc4985f625a"
 					(reference "JP1")

Commit message: layout
Parts:
- JP1, JP2, JP3: footprint Jumper:SolderJumper-2_P1.3mm_Open_TrianglePad1.0x1.5mm -> Resistor_SMD:R_0402_1005Metric
Changed lines of the file:
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@@
 			)
 		)
-		(property "Footprint" "Jumper:SolderJumper-2_P1.3mm_Open_TrianglePad1.0x1.5mm"
+		(property "Footprint" "Resistor_SMD:R_0402_1005Metric"
 			(at 140.97 53.34 0)
 			(effects
@@
 			)
 		)
-		(property "Footprint" "Jumper:SolderJumper-2_P1.3mm_Open_TrianglePad1.0x1.5mm"
+		(property "Footprint" "Resistor_SMD:R_0402_1005Metric"
 			(at 158.75 53.34 0)
 			(effects
@@
 			)
 		)
-		(property "Footprint" "Jumper:SolderJumper-2_P1.3mm_Open_TrianglePad1.0x1.5mm"
+		(property "Footprint" "Resistor_SMD:R_0402_1005Metric"
 			(at 123.19 53.34 0)
 			(effects

Commit message: layout done
Parts:
- R20, R21, R35: value 0.001R -> 0.003R
Changed lines of the file:
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@@
 			)
 		)
-		(property "Value" "0.001R"
+		(property "Value" "0.003R"
 			(at 139.446 45.974 0)
 			(effects
@@
 			)
 		)
-		(property "Value" "0.001R"
+		(property "Value" "0.003R"
 			(at 121.412 45.72 0)
 			(effects
@@
 			)
 		)
-		(property "Value" "0.001R"
+		(property "Value" "0.003R"
 			(at 157.734 45.72 0)
 			(effects
