File: ESC_PCB/ESC_3S/ESC_3S.kicad_pcb (KiCad board)
At the start: 2 copper layers, 117 parts, among them J1 DEBUG&FLASH, J2 Conn_01x01_Pin, J3 Conn_01x01_Pin, J4 Conn_01x04_Pin, J5 UART, J6 U, J7 V, J8 W, Q1 CSD18532Q5BT, Q2 CSD18532Q5BT, Q3 CSD18532Q5BT, Q4 CSD18532Q5BT, Q5 CSD18532Q5BT, Q6 CSD18532Q5BT, U1 MIC5219-3.3YM5, U2 MP2359, U3 STM32G431CBUx, U4 FD6288Q, U5 SN65HVD230DR, X1 Q13FC1350000400, X2 X50328MSB2GI

Commit message: dang layout
Parts:
- C10, C11, C12, C13, C14, C15, C16, C17, C18, C39, C40, C41, C43, C7, C8, C9, D2, D3, D4, D6, D7, FB1, R20, R21, R22, R23, R24, R25, R26, R27, R3, R31, R32, R33, R34, R35, R36, R37, R38, R4, S1, S2, U3, U4, U5, X1, X2: moved to B.Cu
- moved R33 84.9 mm to (145.2, 57.5), turned to 90 degrees
- moved J4 83.7 mm to (149.8, 64.6), turned to 180 degrees
- moved R32 83.6 mm to (145.2, 63.5), turned to -90 degrees
- moved C43 78.5 mm to (125.8, 104.5), turned to 180 degrees
- moved D7 75.4 mm to (146.7, 57.5), turned to 90 degrees
- moved D6 74.3 mm to (146.7, 63.5), turned to -90 degrees
- moved U5 73.6 mm to (139.9, 60.3), turned to 90 degrees
- moved R31 73.4 mm to (135.1, 63.3), turned to -90 degrees
- moved R34 72.5 mm to (132.6, 60.3), turned to 90 degrees
- moved FB1 62.2 mm to (113.8, 63.8)
- moved C12 59.2 mm to (116.7, 63.8), turned to 90 degrees
- moved C15 58.6 mm to (113.8, 67.2), turned to -90 degrees
- moved C16 56.1 mm to (116.8, 67.2), turned to -90 degrees
- moved C17 55.2 mm to (115.3, 67.2), turned to -90 degrees
- moved U3 48.4 mm to (121.7, 67.0), turned to 90 degrees
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Routing:
- net /Gate Driver and 3PH Inverter Bridge/TIM1_CH3N: track 0.00 -> 7.19 mm
- net Net-(D2-K): track 0.00 -> 4.70 mm
Other:
- board outline added: 51.5 x 35 mm

Commit message: layout
Parts:
- removed J1: DEBUG&FLASH, Connector_PinHeader_2.54mm:PinHeader_1x05_P2.54mm_Vertical
- added U6: SM04B-GHS-TB, easyeda2kicad:CONN-SMD_4P-P1.25_SM04B-GHS-TB-LF-SN, B.Cu at (126.4, 79.6)
- C1, C19, C2, C20, C21, C3, C4, C42, J5, L1, R1, R2, R28, U2: moved to B.Cu
- C43, R20, R21, R22, R23, R24, R25, R26, R27, R35, R36, R37, R38: moved to F.Cu
- J4: value Conn_01x04_Pin -> Flash&Debug; footprint Connector_PinHeader_2.54mm:PinHeader_1x04_P2.54mm_Vertical -> Connector_PinHeader_1.27mm:PinHeader_1x04_P1.27mm_Vertical
- JP1, JP2, JP3: footprint Jumper:SolderJumper-2_P1.3mm_Open_TrianglePad1.0x1.5mm -> Resistor_SMD:R_0402_1005Metric; moved to B.Cu
- moved J5 90.9 mm to (157.5, 64.7), turned to 180 degrees
- moved D5 82.2 mm to (172.7, 89.1)
- moved R29 82.2 mm to (168.6, 88.1)
- moved R30 82.2 mm to (168.6, 89.6)
- moved L1 79.3 mm to (91.5, 68.0), turned to 90 degrees
- moved C1 78.8 mm to (94.3, 71.5), turned to 180 degrees
- moved R3 76.9 mm to (73.9, 69.0), turned to 0 degrees
- moved C2 76.6 mm to (91.0, 71.5), turned to 180 degrees
- moved C4 75.5 mm to (94.0, 62.8), turned to 180 degrees
- moved C11 74.7 mm to (73.9, 70.5), turned to 180 degrees
- moved U2 74.0 mm to (94.2, 68.0), turned to 90 degrees
- moved R2 71.9 mm to (92.2, 64.5)
- moved S1 68.5 mm to (75.2, 73.7), turned to 180 degrees
- moved C3 66.6 mm to (96.5, 67.6), turned to 90 degrees
- moved U1 66.5 mm to (120.1, 72.5)
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Connections:
- J4 pad 1: +3.3V -> GND
- J4 pad 2: GND -> /MCU Section/SWDIO
- J4 pad 3: /Addition/CAN_H -> /MCU Section/SWCLK
- J4 pad 4: /Addition/CAN_L -> /MCU Section/SWO
Routing:
- net /Gate Driver and 3PH Inverter Bridge/Curr_fdbk1_OPAmp+: track 0.00 -> 29.8 mm, vias 0 -> 1
- net GND: track 0.00 -> 27.3 mm
- net +9V: track 0.00 -> 23.2 mm
- net /Addition/CAN_RX: track 0.00 -> 21.7 mm, vias 0 -> 2
- net /Gate Driver and 3PH Inverter Bridge/Curr_fdbk2_OPAmp+: track 0.00 -> 19.0 mm, vias 0 -> 1
- net /Gate Driver and 3PH Inverter Bridge/V_Shunt_3+: track 0.00 -> 18.5 mm, vias 0 -> 2
- net /Addition/CAN_L: track 0.00 -> 18.1 mm
- net Net-(D3-K): track 0.00 -> 16.7 mm
- net /MCU Section/BOOT0: track 0.00 -> 16.3 mm
- net /Addition/CAN_H: track 0.00 -> 16.2 mm
- net /Gate Driver and 3PH Inverter Bridge/TIM1_CH1: track 0.00 -> 13.0 mm, vias 0 -> 2
- net /MCU Section/OSC_OUT: track 0.00 -> 12.2 mm
- net Net-(U2-BS): track 0.00 -> 11.9 mm
- net /Gate Driver and 3PH Inverter Bridge/TIM1_CH2: track 0.00 -> 11.2 mm, vias 0 -> 2
- net +3.3V: track 0.00 -> 11.1 mm
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Other:
- board size 51.5 x 35 mm -> 51.5 x 41 mm

Commit message: layout done
Parts:
- removed C5: 2.2uF 16V, Capacitor_SMD:C_1206_3216Metric_Pad1.33x1.80mm_HandSolder
- removed J5: UART, Connector_PinHeader_2.54mm:PinHeader_1x04_P2.54mm_Vertical
- removed U1: MIC5219-3.3YM5, Package_TO_SOT_SMD:SOT-23-5
- added C44: 100nF 25V, Capacitor_SMD:C_0603_1608Metric_Pad1.08x0.95mm_HandSolder, F.Cu at (114.3, 158.3)
- added C45: 100nF, Capacitor_SMD:C_0603_1608Metric_Pad1.08x0.95mm_HandSolder, F.Cu at (129.3, 158.1)
- added D8: SS34, Diode_SMD:D_SMA_Handsoldering, F.Cu at (120.4, 156.3)
- added J1: UART, Connector_PinHeader_1.27mm:PinHeader_1x03_P1.27mm_Vertical, F.Cu at (103.4, 135.9)
- added U7: LD1117S33TR_SOT223, Package_TO_SOT_SMD:SOT-223-3_TabPin2, F.Cu at (131.6, 153.7)
- C1: value 22pF 25V -> 10nF 25V; moved to F.Cu
- C10, C11, C12, C13, C14, C15, C16, C17, C18, C19, C2, C20, C21, C3, C39, C4, C40, C41, C42, C7, C8, C9, D2, D3, D4, D6, D7, FB1, JP1, JP2, JP3, L1, R1, R2, R28, R3, R31, R32, R33, R4, S1, S2, U2, U3, U4, U5, X1, X2: moved to F.Cu
- C43, D5, R22, R23, R24, R25, R26, R27, R29, R30, R36, R37, R38, TH1: moved to B.Cu
- C6: value 470pF -> 10uF
- R20, R21, R35: value 0.001R -> 0.003R; moved to B.Cu
- moved R2 93.5 mm to (105.8, 157.0), turned to 0 degrees
- moved R29 93.5 mm to (103.2, 154.8), turned to 90 degrees
- moved C11 93.3 mm to (131.0, 144.3), turned to -90 degrees
- moved C33 92.3 mm to (129.0, 165.3), turned to -90 degrees
- moved C4 91.8 mm to (116.4, 151.7), turned to -90 degrees
- moved R3 91.8 mm to (131.0, 140.8), turned to -90 degrees
- moved C34 91.4 mm to (127.5, 165.3), turned to -90 degrees
- moved J3 91.3 mm to (105.4, 165.2), turned to 180 degrees
- moved D1 90.7 mm to (132.1, 165.4), turned to -90 degrees
- moved C35 90.7 mm to (126.0, 165.3), turned to -90 degrees
- moved U2 90.4 mm to (109.9, 157.0), turned to 180 degrees
- moved R1 90.1 mm to (105.8, 154.0)
- moved C25 90.0 mm to (124.5, 165.3), turned to -90 degrees
- moved C24 89.4 mm to (123.0, 165.3), turned to -90 degrees
- moved C23 89.0 mm to (121.5, 165.3), turned to -90 degrees
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Connections:
- C6 pad 1: Net-(U1-BP) -> +3.3V
Routing:
- net /Gate Driver and 3PH Inverter Bridge/V_Shunt_2-: track 5.11 -> 69.6 mm
- net /Gate Driver and 3PH Inverter Bridge/V_Shunt_1-: track 5.51 -> 62.7 mm, vias 0 -> 2
- net /Gate Driver and 3PH Inverter Bridge/V_Shunt_1+: track 3.51 -> 51.3 mm, vias 0 -> 1
- net /Gate Driver and 3PH Inverter Bridge/V_Shunt_3-: track 5.88 -> 50.6 mm, vias 0 -> 2
- net /Gate Driver and 3PH Inverter Bridge/V_Shunt_2+: track 0.00 -> 43.6 mm, vias 0 -> 1
- net +3.3V: track 11.1 -> 53.9 mm, vias 0 -> 2
- net /Gate Driver and 3PH Inverter Bridge/Phase_1: track 3.80 -> 38.4 mm, vias 0 -> 2
- net Net-(Q6-G): track 3.70 -> 36.8 mm
- net /Gate Driver and 3PH Inverter Bridge/TIM1_CH1N: track 7.02 -> 30.0 mm, vias 1 -> 2
- net GND: track 27.3 -> 6.53 mm, vias 0 -> 3
- net /Gate Driver and 3PH Inverter Bridge/Phase_3: track 1.95 -> 22.4 mm, vias 0 -> 2
- net /Gate Driver and 3PH Inverter Bridge/Curr_fdbk1_OPAmp+: track 29.8 -> 9.78 mm
- net Net-(Q2-G): track 3.68 -> 23.6 mm, vias 0 -> 2
- net /Gate Driver and 3PH Inverter Bridge/HO1: track 0.00 -> 19.9 mm
- net /Gate Driver and 3PH Inverter Bridge/V_Shunt_3+: track 18.5 -> 37.2 mm, vias 2 -> 1
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Other:
- board size 51.5 x 41 mm -> 40 x 84.6 mm

Commit message: xuat gerber done
Parts:
- moved R29 0.20 mm to (103.0, 154.8)
- renumbered J2 to BAT+, J3 to BAT-, J4 to FLASH, J1 to UART
Routing:
- net +9V: track 11.5 -> 99.5 mm, vias 0 -> 4
- net +3.3V: track 53.9 -> 127.7 mm, vias 2 -> 4
- net GND: track 6.53 -> 56.8 mm, vias 3 -> 39
- net /Addition/VBAT_SENS: track 18.3 -> 35.3 mm
- net +BATT: track 0.00 -> 10.4 mm, vias 0 -> 24
- net /Addition/CAN_RX: track 30.7 -> 35.1 mm
- net Net-(Q2-G): track 23.6 -> 27.5 mm
- net /Gate Driver and 3PH Inverter Bridge/HO3: track 6.40 -> 5.40 mm
- net /Gate Driver and 3PH Inverter Bridge/V_Shunt_2-: track 69.6 -> 70.2 mm, vias 0 -> 2
- net /Gate Driver and 3PH Inverter Bridge/V_Shunt_3+: vias 1 -> 2
- net /Gate Driver and 3PH Inverter Bridge/V_Shunt_2+: vias 1 -> 2
- net /Gate Driver and 3PH Inverter Bridge/V_Shunt_1+: vias 1 -> 2
- added copper zone on B.Cu, net GND
- added copper zone on F.Cu, net GND
Other:
- board size 40 x 84.6 mm -> 40 x 81.7 mm
